Commit message: Imported upstream version '1.1.3' of 'upstream'

File: summit_xl_description/urdf/bases/summit_xl_base.gazebo.xacro (robot description, xacro)
@@ -5,6 +5,6 @@
     <gazebo>
       <plugin name="ros_control" filename="libgazebo_ros_control.so">
-        <robotNamespace>/summit_xl</robotNamespace>
-        <robotParam>robot_description</robotParam>
+        <!--<robotNamespace>/summit_xl</robotNamespace>-->
+		<robotParam>robot_description</robotParam>
         <controlPeriod>0.001</controlPeriod>
 	    <robotSimType>gazebo_ros_control/DefaultRobotHWSim</robotSimType>
@@ -13,49 +13,50 @@
 	</xacro:macro>
 	<!-- skid steering plugin -->
-	<xacro:macro name="skid_steering" params="broadcastOdomTF">
+	<xacro:macro name="skid_steering" params="broadcastOdomTF prefix">
     <gazebo>
       <plugin name="skid_steer_drive_controller" filename="libgazebo_ros_skid_steer_drive.so">
-			<robotNamespace>/summit_xl</robotNamespace>
+			<!--<robotNamespace>/summit_xl</robotNamespace>-->
 		    <updateRate>100.0</updateRate>
-		    <leftFrontJoint>joint_front_left_wheel</leftFrontJoint>
-		    <rightFrontJoint>joint_front_right_wheel</rightFrontJoint>
-		    <leftRearJoint>joint_back_left_wheel</leftRearJoint>
-		    <rightRearJoint>joint_back_right_wheel</rightRearJoint>
+		    <leftFrontJoint>${prefix}joint_front_left_wheel</leftFrontJoint>
+		    <rightFrontJoint>${prefix}joint_front_right_wheel</rightFrontJoint>
+		    <leftRearJoint>${prefix}joint_back_left_wheel</leftRearJoint>
+		    <rightRearJoint>${prefix}joint_back_right_wheel</rightRearJoint>
 		    <!-- wheelSeparation>0.566</wheelSeparation --> <!-- real parameter value -->
 		    <wheelSeparation>1.5</wheelSeparation> <!-- works a bit better in Gazebo -->
 		    <wheelDiameter>0.234</wheelDiameter>
-		    <robotBaseFrame>base_footprint</robotBaseFrame>
+		    <robotBaseFrame>${prefix}base_footprint</robotBaseFrame>
 		    <torque>50</torque>
-		    <commandTopic>/summit_xl_control/cmd_vel</commandTopic>
-		    <odometryTopic>odom</odometryTopic>
-		    <odometryFrame>/odom</odometryFrame>
+		    <commandTopic>robotnik_base_control/cmd_vel</commandTopic>
+		    <odometryTopic>robotnik_base_control/odom</odometryTopic>
+		    <!--odometryFrame>/odom</odometryFrame-->
+		    <odometryFrame>${prefix}odom</odometryFrame>
 		    <broadcastTF>${broadcastOdomTF}</broadcastTF>
       </plugin>
     </gazebo>
   </xacro:macro>
-  <xacro:macro name="omni_steering">
+  <xacro:macro name="omni_steering" params="prefix publish_tf">
 		<gazebo>
 	    <plugin name="omni_steering" filename="libgazebo_ros_planar_move.so">
-	      <commandTopic>/summit_xl_control/cmd_vel</commandTopic>
-	      <odometryTopic>/summit_xl/odom</odometryTopic>
-	      <odometryFrame>odom</odometryFrame>
-	      <odometryRate>20.0</odometryRate>
-	      <robotBaseFrame>base_footprint</robotBaseFrame>
+	      <commandTopic>robotnik_base_control/cmd_vel</commandTopic>
+	      <odometryTopic>robotnik_base_control/odom</odometryTopic>
+	      <odometryFrame>${prefix}odom</odometryFrame>
+	      <odometryRate>50.0</odometryRate>
+	      <robotBaseFrame>${prefix}base_footprint</robotBaseFrame>
+	      <publishTF>${publish_tf}</publishTF>
 	    </plugin>
 	  </gazebo>
   </xacro:macro>
-  <xacro:macro name="ros_force_based_move" params="broadcastOdomTF">
+  <xacro:macro name="ros_force_based_move" params="publish_tf prefix">
 	  <gazebo>
 		 <plugin name="ros_force_based_move" filename="libgazebo_ros_force_based_move.so">
-			 <robotNamespace>/summit_xl</robotNamespace>
-			 <commandTopic>/summit_xl_control/cmd_vel</commandTopic>
-			 <odometryTopic>/summit_xl/odom</odometryTopic>
-	         <odometryFrame>odom</odometryFrame>
+			 <commandTopic>robotnik_base_control/cmd_vel</commandTopic>
+			 <odometryTopic>robotnik_base_control/odom</odometryTopic>
+	         <odometryFrame>${prefix}odom</odometryFrame>
 			 <yaw_velocity_p_gain>10000.0</yaw_velocity_p_gain>
 			 <x_velocity_p_gain>10000.0</x_velocity_p_gain>
 			 <y_velocity_p_gain>10000.0</y_velocity_p_gain>
-			 <robotBaseFrame>base_footprint</robotBaseFrame>
-			 <odometryRate>20.0</odometryRate>
-			 <publishOdometryTf>${broadcastOdomTF}</publishOdometryTf>
+			 <robotBaseFrame>${prefix}base_footprint</robotBaseFrame>
+			 <odometryRate>50.0</odometryRate>
+			 <publishOdometryTf>${publish_tf}</publishOdometryTf>
 		 </plugin>
 	  </gazebo>

File: summit_xl_description/urdf/bases/summit_xl_base.urdf.xacro (robot description, xacro)
@@ -2,54 +2,54 @@
 <robot name="summit_xl" xmlns:xacro="http://www.ros.org/wiki/xacro">
   <xacro:include filename="$(find summit_xl_description)/urdf/bases/summit_xl_base.gazebo.xacro" />
-  <xacro:macro name="summit_xl_base" params="name publish_bf hq">
-  <!-- Robot mechanical and motor parameters -->
-  <xacro:property name="PI" value="3.1415926535897931"/>
-  <xacro:property name="wheel_width" value="0.175" />
-  <!-- BASE FOOTPRINT -->
-  <xacro:if value="${publish_bf}">
-    <link name="base_footprint">
-      <visual>
-          <origin xyz="0 0 0" rpy="0 0 0" />
-          <geometry>
-             <box size="0.001 0.001 0.001" />
-          </geometry>
-      </visual>
-    </link>
-    <joint name="base_footprint_joint" type="fixed">
-      <origin xyz="0 0 ${wheel_radius}" rpy="0 0 0" /> <!-- ${wheel_radius} property must be defined inside wheel description -->
-      <parent link="base_footprint"/>
-      <child link="base_link" />
-    </joint>
-  </xacro:if>
-  <!-- BASE_LINK -->
-  <link name="base_link">
-    <inertial>
-      <mass value="25.0" />
-      <origin xyz="0 0 0" />
-      <inertia  ixx="1.391" ixy="0.004"  ixz="0.0"  iyy="6.853"  iyz="0.0"  izz="6.125" />
-    </inertial>
-    <visual>
-       <origin xyz="0 0 0" rpy="0 0 0" />
-       <xacro:if value="${hq}">
-       <geometry>
-	     <mesh filename="package://summit_xl_description/meshes/bases/summit_xl_chassis.dae"/>
-       </geometry>
-       </xacro:if>
-       <xacro:unless value="${hq}">
-       <geometry>
-	     <mesh filename="package://summit_xl_description/meshes/bases/summit_xl_chassis_simple.stl"/>
-       </geometry>
-       </xacro:unless>
-       <material name="darkgrey">
-         <color rgba="0.1 0.1 0.1 1"/>
-       </material>
-    </visual>
-    <collision>
-       <origin xyz="0 0 0" rpy="0 0 0 " />
-       <geometry>
-         <mesh filename="package://summit_xl_description/meshes/bases/summit_xl_chassis_collision.dae"/>
-       </geometry>
-    </collision>
-  </link>
+  <xacro:macro name="summit_xl_base" params="prefix publish_bf hq">
+	  <!-- Robot mechanical and motor parameters -->
+	  <xacro:property name="PI" value="3.1415926535897931"/>
+	  <xacro:property name="wheel_width" value="0.175" />
+	  <!-- BASE FOOTPRINT -->
+	  <xacro:if value="${publish_bf}">
+		<link name="${prefix}base_footprint">
+		  <visual>
+			  <origin xyz="0 0 0" rpy="0 0 0" />
+			  <geometry>
+				 <box size="0.001 0.001 0.001" />
+			  </geometry>
+		  </visual>
+		</link>
+		<joint name="${prefix}base_footprint_joint" type="fixed">
+		  <origin xyz="0 0 ${wheel_radius}" rpy="0 0 0" /> <!-- ${wheel_radius} property must be defined inside wheel description -->
+		  <parent link="${prefix}base_footprint"/>
+		  <child link="${prefix}base_link" />
+		</joint>
+	  </xacro:if>
+	  <!-- BASE_LINK -->
+	  <link name="${prefix}base_link">
+		<inertial>
+		  <mass value="25.0" />
+		  <origin xyz="0 0 0" />
+		  <inertia  ixx="1.391" ixy="0.004"  ixz="0.0"  iyy="6.853"  iyz="0.0"  izz="6.125" />
+		</inertial>
+		<visual>
+		   <origin xyz="0 0 0" rpy="0 0 0" />
+		   <xacro:if value="${hq}">
+		   <geometry>
+			 <mesh filename="package://summit_xl_description/meshes/bases/summit_xl_chassis.dae"/>
+		   </geometry>
+		   </xacro:if>
+		   <xacro:unless value="${hq}">
+		   <geometry>
+			 <mesh filename="package://summit_xl_description/meshes/bases/summit_xl_chassis_simple.stl"/>
+		   </geometry>
+		   </xacro:unless>
+		   <material name="darkgrey">
+			 <color rgba="0.1 0.1 0.1 1"/>
+		   </material>
+		</visual>
+		<collision>
+		   <origin xyz="0 0 0" rpy="0 0 0 " />
+		   <geometry>
+			 <mesh filename="package://summit_xl_description/meshes/bases/summit_xl_chassis_collision.dae"/>
+		   </geometry>
+		</collision>
+	  </link>
   </xacro:macro>
 </robot>

File: summit_xl_description/urdf/bases/summit_xl_hls_base.urdf.xacro (robot description, xacro)
@@ -2,28 +2,28 @@
 <robot name="summit_xl" xmlns:xacro="http://www.ros.org/wiki/xacro">
   <xacro:include filename="$(find summit_xl_description)/urdf/bases/summit_xl_base.gazebo.xacro" />
-  <xacro:macro name="summit_xl_hls_base" params="name publish_bf hq">
-  <!-- Robot mechanical and motor parameters -->
-  <xacro:property name="PI" value="3.1415926535897931"/>
-  <!-- xacro:property name="wheel_width" value="0.175" / -->
-  <!-- BASE FOOTPRINT -->
-  <xacro:if value="${publish_bf}">
-    <link name="base_footprint">
-      <visual>
-          <origin xyz="0 0 0" rpy="0 0 0" />
-          <geometry>
-             <box size="0.001 0.001 0.001" />
-          </geometry>
-      </visual>
-    </link>
-    <joint name="base_footprint_joint" type="fixed">
-      <origin xyz="0 0 ${wheel_radius}" rpy="0 0 0" /> <!-- ${wheel_radius} property must be defined inside wheel description -->
-      <parent link="base_footprint"/>
-      <child link="base_link" />
-    </joint>
-  </xacro:if>
+  <xacro:macro name="summit_xl_hls_base" params="prefix publish_bf hq">
+	  <!-- Robot mechanical and motor parameters -->
+	  <xacro:property name="PI" value="3.1415926535897931"/>
+	  <xacro:property name="wheel_width" value="0.175" />
+	<!-- BASE FOOTPRINT -->
+	  <xacro:if value="${publish_bf}">
+		<link name="${prefix}base_footprint">
+		  <visual>
+			  <origin xyz="0 0 0" rpy="0 0 0" />
+			  <geometry>
+				 <box size="0.001 0.001 0.001" />
+			  </geometry>
+		  </visual>
+		</link>
+		<joint name="${prefix}base_footprint_joint" type="fixed">
+		  <origin xyz="0 0 ${wheel_radius}" rpy="0 0 0" /> <!-- ${wheel_radius} property must be defined inside wheel description -->
+		  <parent link="${prefix}base_footprint"/>
+		  <child link="${prefix}base_link" />
+		</joint>
+	  </xacro:if>
   <!-- BASE_LINK -->
-  <link name="base_link">
+  <link name="${prefix}base_link">
     <inertial>
-      <mass value="25.0" />
+      <mass value="125.0" />
       <origin xyz="0 0 0" />
       <inertia  ixx="1.391" ixy="0.004"  ixz="0.0"  iyy="6.853"  iyz="0.0"  izz="6.125" />
@@ -52,4 +52,12 @@
     </collision>
   </link>
+   <!-- DOCKING CONTACT -->
+    <link name="${prefix}base_docking_contact">
+    </link>
+    <joint name="${prefix}base_docking_joint" type="fixed">
+      <origin xyz="0.30 0 0.09" rpy="0 0 0" />
+      <parent link="${prefix}base_link"/>
+      <child link="${prefix}base_docking_contact" />
+    </joint>
   </xacro:macro>
 </robot>

File: summit_xl_description/urdf/wheels/omni_wheel.urdf.xacro (robot description, xacro)
@@ -8,11 +8,11 @@
   <xacro:macro name="cylinder_inertia" params="m r h">
     <inertia  ixx="${m*(3*r*r+h*h)/12}" ixy = "0" ixz = "0"
-              iyy="${m*(3*r*r+h*h)/12}" iyz = "0"
-              izz="${m*r*r/2}" />
+              iyy="${m*r*r/2}" iyz = "0"
+              izz="${m*(3*r*r+h*h)/12}" />
   </xacro:macro>
-  <xacro:macro name="omni_wheel" params="name parent *origin reflect hq">
-    <joint name="joint_${name}_wheel" type="continuous">
+  <xacro:macro name="omni_wheel" params="prefix parent *origin reflect hq">
+    <joint name="${prefix}_wheel_joint" type="continuous">
       <parent link="${parent}"/>
-      <child link="${name}_wheel"/>
+      <child link="${prefix}_wheel_link"/>
       <xacro:insert_block name="origin" />
       <axis xyz="0 1 0" rpy="0 0 0" />
@@ -20,5 +20,5 @@
       <joint_properties damping="0.0" friction="0.0"/>
     </joint>
-    <link name="${name}_wheel">
+    <link name="${prefix}_wheel_link">
       <visual>
         <xacro:if value="${hq}">
@@ -33,5 +33,5 @@
               <mesh filename="package://summit_xl_description/meshes/wheels/omni_wheel_2.dae" />
             </geometry>
-		  s</xacro:unless>
+		  </xacro:unless>
         </xacro:if>
         <xacro:unless value="${hq}">
@@ -69,14 +69,14 @@
     </link>
     <!-- Transmission is important to link the joints and the controller (see summit_xl_control/config/summit_xl_control.yaml)-->
-    <transmission name="${name}_wheel_joint_trans">
+    <transmission name="${prefix}_wheel_joint_trans">
       <type>transmission_interface/SimpleTransmission</type>
-      <joint name="joint_${name}_wheel" >
-         <hardwareInterface>EffortJointInterface</hardwareInterface>
+      <joint name="${prefix}_wheel_joint" >
+        <hardwareInterface>hardware_interface/VelocityJointInterface</hardwareInterface>
       </joint>
-      <actuator name="${name}_wheel_joint_motor">
+      <actuator name="${prefix}_wheel_joint_motor">
          <mechanicalReduction>1</mechanicalReduction>
       </actuator>
     </transmission>
-    <gazebo reference="${name}_wheel">
+    <gazebo reference="${prefix}_wheel_link">
 		<mu1 value="1.0"/>
 		<mu2 value="1.0"/>

File: summit_xl_description/urdf/wheels/rubber_wheel.urdf.xacro (robot description, xacro)
@@ -3,17 +3,17 @@
   <xacro:property name="M_PI" value="3.1415926535897931" />
   <!-- Wheels -->
-  <xacro:property name="wheel_radius" value="0.117" />
-  <xacro:property name="wheel_height" value="0.14" />
+  <xacro:property name="wheel_radius" value="0.125" />
+  <xacro:property name="wheel_height" value="0.14" /> <!-- really is the wheel width -->
   <xacro:property name="wheel_mass" value="6.5" /> <!-- in kg-->
   <xacro:macro name="cylinder_inertia" params="m r h">
     <inertia  ixx="${m*(3*r*r+h*h)/12}" ixy = "0" ixz = "0"
-              iyy="${m*(3*r*r+h*h)/12}" iyz = "0"
-              izz="${m*r*r/2}" />
+              iyy="${m*r*r/2}" iyz = "0"
+              izz="${m*(3*r*r+h*h)/12}" />
   </xacro:macro>
-  <xacro:macro name="rubber_wheel" params="name parent *origin reflect hq">
+  <xacro:macro name="rubber_wheel" params="prefix parent *origin reflect hq">
 <!--WHEEL TIRE -->
-    <joint name="joint_${name}_wheel" type="continuous">
+    <joint name="${prefix}_wheel_joint" type="continuous">
       <parent link="${parent}"/>
-      <child link="${name}_wheel"/>
+      <child link="${prefix}_wheel"/>
       <xacro:insert_block name="origin" />
       <axis xyz="0 1 0" rpy="0 0 0" />
@@ -21,5 +21,5 @@
       <joint_properties damping="0.0" friction="0.0"/>
     </joint>
-    <link name="${name}_wheel">
+    <link name="${prefix}_wheel">
       <visual>
         <!-- HIGH RESOLUTION WHEELS -->
@@ -56,14 +56,15 @@
     </link>
     <!-- Transmission is important to link the joints and the controller (see summit_xl_control/config/summit_xl_control.yaml)-->
-    <transmission name="${name}_wheel_joint_trans">
+    <transmission name="${prefix}_wheel_joint_trans">
       <type>transmission_interface/SimpleTransmission</type>
-      <joint name="joint_${name}_wheel">
-		<hardwareInterface>EffortJointInterface</hardwareInterface>
+      <joint name="${prefix}_wheel_joint">
+        <hardwareInterface>hardware_interface/VelocityJointInterface</hardwareInterface>
       </joint>
-      <actuator name="${name}_wheel_joint_motor">
+      <actuator name="${prefix}_wheel_joint_motor">
         <mechanicalReduction>1</mechanicalReduction>
+        <motorTorqueConstant>20</motorTorqueConstant>
       </actuator>
      </transmission>
-    <gazebo reference="${name}_wheel">
+    <gazebo reference="${prefix}_wheel">
 			<mu1 value="1.0"/>
 			<mu2 value="1.0"/>
