Commit message: Rebase from 'release/kinetic/summit_xl_description'

File: robots/summit_xl_std.urdf.xacro (robot description, xacro)
@@ -19,4 +19,5 @@
 	<xacro:property name="hq" value="true" />
 	<xacro:arg name="prefix" default="summit_xl_"/>
+	<xacro:arg name="ros_planar_move_plugin" default="false"/>
     <xacro:macro name="summit_xl" params="prefix publish_bf hq">
 		<!-- *************** -->
@@ -38,26 +39,30 @@
 			<origin xyz="-${wheel_offset_x} -${wheel_offset_y} ${wheel_offset_z}" rpy="0 0 0"/>
 		</xacro:rubber_wheel>
+        <!-- IMU -->
 		<xacro:sensor_imu_hector prefix="$(arg prefix)imu" parent="$(arg prefix)base_link">
 			<origin xyz="-0.18 0.0 0.170" rpy="0 0 0"/>
 		</xacro:sensor_imu_hector>
 		<!-- 2d laser -->
-		<!--xacro:sensor_hokuyo_ust10lx prefix="$(arg prefix)front_laser" parent="$(arg prefix)base_link" prefix_topic="front_laser">
+		<xacro:sensor_hokuyo_ust10lx prefix="$(arg prefix)front_laser" parent="$(arg prefix)base_link" prefix_topic="front_laser">
 			<origin xyz="0.0 0.0 0.33" rpy="0 0 0"/>
-		</xacro:sensor_hokuyo_ust10lx-->
+		</xacro:sensor_hokuyo_ust10lx>
 		<!-- ptz camera -->
-		<!--xacro:sensor_axis prefix="$(arg prefix)front_ptz_camera" parent="$(arg prefix)base_link">
+		<xacro:sensor_axis prefix="$(arg prefix)front_ptz_camera" parent="$(arg prefix)base_link">
 			<origin xyz="0.19 0 0.26" rpy="0 ${15*PI/180} 0"/>
-		</xacro:sensor_axis-->
+		</xacro:sensor_axis>
 	    <!-- RGBD -->
-	    <!--xacro:sensor_orbbec_astra prefix="$(arg prefix)front_rgbd_camera" parent="$(arg prefix)base_link" prefix_topic="front_rgbd_camera">
+	    <xacro:sensor_orbbec_astra prefix="$(arg prefix)front_rgbd_camera" parent="$(arg prefix)base_link" prefix_topic="front_rgbd_camera">
 			<origin xyz="0.324 0.012 0.172" rpy="0 0 0"/>
-		</xacro:sensor_orbbec_astra-->
+		</xacro:sensor_orbbec_astra>
 	    <!-- GPS -->
-	    <!--xacro:sensor_gps prefix="$(arg prefix)gps" parent="$(arg prefix)base_link">
+	    <xacro:sensor_gps prefix="$(arg prefix)gps" parent="$(arg prefix)base_link">
 			<origin xyz="-0.22 0 0.275" rpy="0 0 0"/>
-		</xacro:sensor_gps-->
+		</xacro:sensor_gps>
    </xacro:macro>
    <!-- Gazebo ros control pluggins -->
    <xacro:ros_control/>
+   <xacro:if value="$(arg ros_planar_move_plugin)">
+	   <xacro:omni_steering prefix="$(arg prefix)" publish_tf="false"/>
+   </xacro:if>
    <xacro:summit_xl prefix="$(arg prefix)" publish_bf="true" hq="true"/>
 </robot>

File: robots/versions/summit_xl_170421A.urdf.xacro (robot description, xacro)
@@ -41,20 +41,12 @@
 			<origin xyz="-0.18 0.0 0.170" rpy="0 0 0"/>
 		</xacro:sensor_imu_hector>
-		<!-- 2d laser -->
-		<!--xacro:sensor_hokuyo_ust10lx prefix="$(arg prefix)front_laser" parent="$(arg prefix)base_link" prefix_topic="front_laser">
+		<!--
+		<xacro:sensor_hokuyo_ust10lx prefix="$(arg prefix)front_laser" parent="$(arg prefix)base_link">
 			<origin xyz="0.0 0.0 0.33" rpy="0 0 0"/>
-		</xacro:sensor_hokuyo_ust10lx-->
-		<!-- ptz camera -->
-		<!--xacro:sensor_axis prefix="$(arg prefix)front_ptz_camera" parent="$(arg prefix)base_link">
-			<origin xyz="0.19 0 0.26" rpy="0 ${15*PI/180} 0"/>
-		</xacro:sensor_axis-->
-	    <!-- RGBD -->
-	    <!--xacro:sensor_orbbec_astra prefix="$(arg prefix)front_rgbd_camera" parent="$(arg prefix)base_link" prefix_topic="front_rgbd_camera">
-			<origin xyz="0.324 0.012 0.172" rpy="0 0 0"/>
-		</xacro:sensor_orbbec_astra-->
-	    <!-- GPS -->
-	    <!--xacro:sensor_gps prefix="$(arg prefix)gps" parent="$(arg prefix)base_link">
-			<origin xyz="-0.22 0 0.275" rpy="0 0 0"/>
-		</xacro:sensor_gps-->
+		</xacro:sensor_hokuyo_ust10lx>
+		-->
+		<xacro:sensor_axis prefix="$(arg prefix)front_ptz_camera" parent="$(arg prefix)base_link">
+			<origin xyz="0.19 0 0.3" rpy="0 ${15*PI/180} 0"/>
+		</xacro:sensor_axis>
    </xacro:macro>
    <!-- Gazebo ros control pluggins -->

File: robots/versions/summit_xl_170518A.urdf.xacro (robot description, xacro)
@@ -42,19 +42,19 @@
 		</xacro:sensor_imu_hector>
 		<!-- 2d laser -->
-		<!--xacro:sensor_hokuyo_ust10lx prefix="$(arg prefix)front_laser" parent="$(arg prefix)base_link" prefix_topic="front_laser">
+		<!--xacro:sensor_hokuyo_ust10lx prefix="$(arg prefix)front_laser" parent="$(arg prefix)base_link">
 			<origin xyz="0.0 0.0 0.33" rpy="0 0 0"/>
 		</xacro:sensor_hokuyo_ust10lx-->
 		<!-- ptz camera -->
-		<!--xacro:sensor_axis prefix="$(arg prefix)front_ptz_camera" parent="$(arg prefix)base_link">
-			<origin xyz="0.19 0 0.26" rpy="0 ${15*PI/180} 0"/>
-		</xacro:sensor_axis-->
+		<xacro:sensor_axis prefix="$(arg prefix)front_ptz_camera" parent="$(arg prefix)base_link">
+			<origin xyz="0.19 0 0.3" rpy="0 ${15*PI/180} 0"/>
+		</xacro:sensor_axis>
 	    <!-- RGBD -->
-	    <!--xacro:sensor_orbbec_astra prefix="$(arg prefix)front_rgbd_camera" parent="$(arg prefix)base_link" prefix_topic="front_rgbd_camera">
+	    <!--xacro:sensor_orbbec_astra prefix="$(arg prefix)front_rgbd_camera" parent="$(arg prefix)base_link">
 			<origin xyz="0.324 0.012 0.172" rpy="0 0 0"/>
 		</xacro:sensor_orbbec_astra-->
 	    <!-- GPS -->
-	    <!--xacro:sensor_gps prefix="$(arg prefix)gps" parent="$(arg prefix)base_link">
+	    <xacro:sensor_gps_with_mast prefix="$(arg prefix)gps" parent="$(arg prefix)base_link">
 			<origin xyz="-0.22 0 0.275" rpy="0 0 0"/>
-		</xacro:sensor_gps-->
+		</xacro:sensor_gps_with_mast>
    </xacro:macro>
    <!-- Gazebo ros control pluggins -->

File: robots/versions/summit_xl_171124A.urdf.xacro (robot description, xacro)
@@ -46,7 +46,7 @@
 		</xacro:sensor_hokuyo_ust10lx-->
 		<!-- ptz camera -->
-		<!--xacro:sensor_axis prefix="$(arg prefix)front_ptz_camera" parent="$(arg prefix)base_link">
+		<xacro:sensor_axis prefix="$(arg prefix)front_ptz_camera" parent="$(arg prefix)base_link">
 			<origin xyz="0.19 0 0.26" rpy="0 ${15*PI/180} 0"/>
-		</xacro:sensor_axis-->
+		</xacro:sensor_axis>
 	    <!-- RGBD -->
 	    <!--xacro:sensor_orbbec_astra prefix="$(arg prefix)front_rgbd_camera" parent="$(arg prefix)base_link" prefix_topic="front_rgbd_camera">

File: urdf/structures/structure_chasis_sup_our.urdf.xacro (robot description, xacro)
@@ -1,5 +1,5 @@
 <?xml version="1.0"?>
-<robot name="structure" xmlns:xacro="http://ros.org/wiki/xacro">
-  <xacro:macro name="structure_ptz" params="prefix parent *origin">
+<robot name="structure" xmlns:xacro="http://www.ros.org/wiki/xacro">
+  <xacro:macro name="structure_chasis_our" params="prefix parent *origin">
 	  <joint name="${prefix}_joint" type="fixed">
 	    <axis xyz="0 1 0"/>
@@ -20,5 +20,5 @@
         </material>
 	      <geometry>
-	        <mesh filename="package://summit_xl_description/meshes/structures/structure_ptz_rgbd_gps.dae"/>
+	        <mesh filename="package://summit_xl_description/meshes/structures/chasis_sup_our.stl"/>
 	      </geometry>
 	    </visual>
@@ -26,5 +26,5 @@
 	      <origin rpy="0 0 0" xyz="0 0 0"/>
 	      <geometry>
-	        <mesh filename="package://summit_xl_description/meshes/structures/structure_ptz_rgbd_gps.dae"/>
+	        <mesh filename="package://summit_xl_description/meshes/structures/chasis_sup_our.stl"/>
 	      </geometry>
 	    </collision>
